File: Ivium Adapter/Ivium Adapter.kicad_pcb (KiCad board)
At the start: 2 copper layers, 49 x 49 mm, 2 parts

Commit message: rB ready... added 20p connect and routed, generated fab files
Parts:
- removed REF**: CON_5034801600_MOL, MOLEX FPC:CON_5034801600_MOL
- removed REF**: JST_SH_BM04B-SRSS-TB_1x04-1MP_P1.00mm_Vertical, Connector_JST:JST_SH_BM04B-SRSS-TB_1x04-1MP_P1.00mm_Vertical
- added ?: , , F.Cu at (117.7, 86.8)
- added ?: , , F.Cu at (115.2, 84.0)
- added ?: , , F.Cu at (119.4, 89.8)
- added ?: , , F.Cu at (112.3, 81.9)
- added J12: 5034802000, 5034802000 FPC Molex:CON_5034802000_MOL, F.Cu at (96.2, 85.9)
- added J6: Qwiic Connect, Connector_JST:JST_SH_BM04B-SRSS-TB_1x04-1MP_P1.00mm_Vertical, B.Cu at (89.3, 81.3)
Routing:
- net SDA: vias 0 -> 1
- net SCL: vias 0 -> 1
- net S2: vias 0 -> 1
- net S1: vias 0 -> 1
- net Heater 1: vias 0 -> 1
- net Heater 0: vias 0 -> 1
- net GND: vias 0 -> 1
- net F2: vias 0 -> 1
- net F1: vias 0 -> 1
- net E5: vias 0 -> 1
- net E4: vias 0 -> 1
- net E3: vias 0 -> 1
- net E2: vias 0 -> 1
- net E1: vias 0 -> 1
- net E0: vias 0 -> 1
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- added copper zone on F.Cu, net GND
Other:
- board text added: "0"
- board text added: "E0"
- board text added: "E1"
- board text added: "E2"
- board text added: "E3"
- board text added: "E4"
- board text added: "E5"
- board text added: "F1"
- board text added: "F2"
- board text added: "H0"
- board text added: "H1"
- board text added: "S1"
- board text added: "S2"
- board text removed: "3"
